Commit message: added calibration tip to franka hand description

File: franka_description/robots/common/franka_hand.xacro (robot description, xacro)
@@ -2,4 +2,6 @@
 <robot xmlns:xacro="http://www.ros.org/wiki/xacro" name="hand">
   <!-- safety_distance: Minimum safety distance in [m] by which the collision volumes are expanded and which is enforced during robot motions -->
+  <!-- Value from measurements and datasheet:-->
+  <xacro:property name="tip_length" value="0.0314" />
   <xacro:macro name="franka_hand" params="connected_to:='' arm_id:='panda' rpy:='0 0 0' xyz:='0 0 0' tcp_xyz:='0 0 0.1034' tcp_rpy:='0 0 0' safety_distance:=0 gazebo:=false description_pkg:=franka_description">
     <xacro:unless value="${connected_to == ''}">
@@ -100,4 +102,23 @@
       </xacro:if>
     </link>
+    <link name="${arm_id}_calibration_needle">
+      <visual>
+        <origin xyz="0 0 ${tip_length/2}" rpy="0 0 0" />
+        <!-- 0.031625 -->
+        <geometry>
+          <cylinder length="${tip_length}" radius="0.001"/>
+        </geometry>
+      </visual>
+      <collision>
+        <origin xyz="0 0 0" rpy="0 0 0" />
+        <geometry>
+          <cylinder length="${tip_length}" radius="0.001"/>
+        </geometry>
+      </collision>
+      <xacro:if value="${gazebo}">
+        <xacro:inertial_props name="calibration_needle" />
+      </xacro:if>
+    </link>
+    <link name="${arm_id}_calibration_tip" />
     <joint name="${arm_id}_finger_joint1" type="prismatic">
       <parent link="${arm_id}_hand" />
@@ -117,4 +138,14 @@
       <dynamics damping="0.3" />
     </joint>
+    <joint name="${arm_id}_cneedle_joint" type="fixed">
+      <parent link="${arm_id}_hand_tcp" />
+      <child link="${arm_id}_calibration_needle" />
+      <origin xyz="0 0 0" rpy="0 0 0" />
+    </joint>
+    <joint name="${arm_id}_ctip_joint" type="fixed">
+      <parent link="${arm_id}_calibration_needle" />
+      <child link="${arm_id}_calibration_tip" />
+      <origin xyz="0 0 ${tip_length} " rpy="0 0 0" />
+    </joint>
   </xacro:macro>
 </robot>
